Commit message: latest commit

File: urdf/robot_arm_old.xacro (robot description, xacro)
@@ -13,5 +13,5 @@
     <origin xyz="0 0 0" rpy="0 0 0"/>
     <geometry>
-      <mesh filename="package://robot_arm_description/meshes/base_link.stl" scale="0.001 0.001 0.001"/>
+      <mesh filename="package://robot_arm_description/meshes/arm_base_link.stl" scale="0.001 0.001 0.001"/>
     </geometry>
     <material name="silver"/>
@@ -20,5 +20,5 @@
     <origin xyz="0 0 0" rpy="0 0 0"/>
     <geometry>
-      <mesh filename="package://robot_arm_description/meshes/base_link.stl" scale="0.001 0.001 0.001"/>
+      <mesh filename="package://robot_arm_description/meshes/arm_base_link.stl" scale="0.001 0.001 0.001"/>
     </geometry>
   </collision>
@@ -46,7 +46,7 @@
 <link name="outaxis1_1">
   <inertial>
-    <origin xyz="0.004045016512831855 3.0931153955585794e-07 1.3540533405891758e-07" rpy="0 0 0"/>
+    <origin xyz="0.004045016512831858 3.093115920902237e-07 1.3540542182118032e-07" rpy="0 0 0"/>
     <mass value="0.03958817250925055"/>
-    <inertia ixx="6e-06" iyy="3e-06" izz="3e-06" ixy="-0.0" iyz="-0.0" ixz="0.0"/>
+    <inertia ixx="6e-06" iyy="3e-06" izz="3e-06" ixy="-0.0" iyz="0.0" ixz="0.0"/>
   </inertial>
   <visual>
@@ -66,10 +66,10 @@
 <link name="fl1_1">
   <inertial>
-    <origin xyz="0.002499770653925492 0.00588930931113294 0.010456135405386759" rpy="0 0 0"/>
+    <origin xyz="0.002499770653925494 -0.0015066906887657814 0.011905135405221725" rpy="0 0 0"/>
     <mass value="0.02382701874556585"/>
     <inertia ixx="4e-06" iyy="2e-06" izz="2e-06" ixy="0.0" iyz="-0.0" ixz="-0.0"/>
   </inertial>
   <visual>
-    <origin xyz="0.00334 0.009339 0.007084" rpy="0 0 0"/>
+    <origin xyz="0.00334 0.001943 0.008533" rpy="0 0 0"/>
     <geometry>
       <mesh filename="package://robot_arm_description/meshes/fl1_1.stl" scale="0.001 0.001 0.001"/>
@@ -78,5 +78,5 @@
   </visual>
   <collision>
-    <origin xyz="0.00334 0.009339 0.007084" rpy="0 0 0"/>
+    <origin xyz="0.00334 0.001943 0.008533" rpy="0 0 0"/>
     <geometry>
       <mesh filename="package://robot_arm_description/meshes/fl1_1.stl" scale="0.001 0.001 0.001"/>
@@ -86,10 +86,10 @@
 <link name="arm1_1">
   <inertial>
-    <origin xyz="0.0024997706539254816 0.004857970392316099 0.10993314740040666" rpy="0 0 0"/>
+    <origin xyz="0.002499770653925497 -0.06164819990760506 0.09114993614509007" rpy="0 0 0"/>
     <mass value="0.15062120277990854"/>
-    <inertia ixx="0.0005" iyy="0.000431" izz="6.9e-05" ixy="0.0" iyz="4e-06" ixz="-0.0"/>
-  </inertial>
-  <visual>
-    <origin xyz="-0.00166 0.009339 0.007084" rpy="0 0 0"/>
+    <inertia ixx="0.0005" iyy="0.000299" izz="0.000201" ixy="0.0" iyz="0.000174" ixz="-0.0"/>
+  </inertial>
+  <visual>
+    <origin xyz="-0.00166 0.001943 0.008533" rpy="0 0 0"/>
     <geometry>
       <mesh filename="package://robot_arm_description/meshes/arm1_1.stl" scale="0.001 0.001 0.001"/>
@@ -98,5 +98,5 @@
   </visual>
   <collision>
-    <origin xyz="-0.00166 0.009339 0.007084" rpy="0 0 0"/>
+    <origin xyz="-0.00166 0.001943 0.008533" rpy="0 0 0"/>
     <geometry>
       <mesh filename="package://robot_arm_description/meshes/arm1_1.stl" scale="0.001 0.001 0.001"/>
@@ -106,10 +106,10 @@
 <link name="motor_2_1">
   <inertial>
-    <origin xyz="0.014068847719958519 0.028626001459861126 0.0003249546058085029" rpy="0 0 0"/>
+    <origin xyz="0.014068847719958543 0.022786589195628024 0.01732961842867156" rpy="0 0 0"/>
     <mass value="0.8439665434293464"/>
-    <inertia ixx="0.000579" iyy="0.000343" izz="0.000355" ixy="0.0" iyz="-0.0" ixz="0.0"/>
-  </inertial>
-  <visual>
-    <origin xyz="-0.00666 0.034052 -0.153054" rpy="0 0 0"/>
+    <inertia ixx="0.000579" iyy="0.000347" izz="0.00035" ixy="0.0" iyz="-6e-06" ixz="0.0"/>
+  </inertial>
+  <visual>
+    <origin xyz="-0.00666 0.117265 -0.105289" rpy="0 0 0"/>
     <geometry>
       <mesh filename="package://robot_arm_description/meshes/motor_2_1.stl" scale="0.001 0.001 0.001"/>
@@ -118,5 +118,5 @@
   </visual>
   <collision>
-    <origin xyz="-0.00666 0.034052 -0.153054" rpy="0 0 0"/>
+    <origin xyz="-0.00666 0.117265 -0.105289" rpy="0 0 0"/>
     <geometry>
       <mesh filename="package://robot_arm_description/meshes/motor_2_1.stl" scale="0.001 0.001 0.001"/>
@@ -126,10 +126,10 @@
 <link name="outaxis2_1">
   <inertial>
-    <origin xyz="-0.004045475204981814 2.594057981128439e-07 -1.4819398216903146e-07" rpy="0 0 0"/>
+    <origin xyz="-0.004045475204981776 4.414634192650979e-07 4.542076181279775e-07" rpy="0 0 0"/>
     <mass value="0.03958817250924634"/>
     <inertia ixx="6e-06" iyy="3e-06" izz="3e-06" ixy="0.0" iyz="0.0" ixz="-0.0"/>
   </inertial>
   <visual>
-    <origin xyz="-0.00766 0.005054 -0.153364" rpy="0 0 0"/>
+    <origin xyz="-0.00766 0.094171 -0.122828" rpy="0 0 0"/>
     <geometry>
       <mesh filename="package://robot_arm_description/meshes/outaxis2_1.stl" scale="0.001 0.001 0.001"/>
@@ -138,5 +138,5 @@
   </visual>
   <collision>
-    <origin xyz="-0.00766 0.005054 -0.153364" rpy="0 0 0"/>
+    <origin xyz="-0.00766 0.094171 -0.122828" rpy="0 0 0"/>
     <geometry>
       <mesh filename="package://robot_arm_description/meshes/outaxis2_1.stl" scale="0.001 0.001 0.001"/>
@@ -146,10 +146,10 @@
 <link name="fl2_1">
   <inertial>
-    <origin xyz="-0.0025002293460745176 0.006111259405306327 -0.010327148194020946" rpy="0 0 0"/>
+    <origin xyz="-0.002500229346074482 0.005899441462926841 -0.010449545792410586" rpy="0 0 0"/>
     <mass value="0.02382701874556588"/>
-    <inertia ixx="4e-06" iyy="2e-06" izz="2e-06" ixy="0.0" iyz="-0.0" ixz="-0.0"/>
-  </inertial>
-  <visual>
-    <origin xyz="0.00034 0.011165 -0.163691" rpy="0 0 0"/>
+    <inertia ixx="4e-06" iyy="2e-06" izz="2e-06" ixy="-0.0" iyz="0.0" ixz="0.0"/>
+  </inertial>
+  <visual>
+    <origin xyz="0.00034 0.10007 -0.133278" rpy="0 0 0"/>
     <geometry>
       <mesh filename="package://robot_arm_description/meshes/fl2_1.stl" scale="0.001 0.001 0.001"/>
@@ -158,5 +158,5 @@
   </visual>
   <collision>
-    <origin xyz="0.00034 0.011165 -0.163691" rpy="0 0 0"/>
+    <origin xyz="0.00034 0.10007 -0.133278" rpy="0 0 0"/>
     <geometry>
       <mesh filename="package://robot_arm_description/meshes/fl2_1.stl" scale="0.001 0.001 0.001"/>
@@ -166,10 +166,10 @@
 <link name="arm2_1">
   <inertial>
-    <origin xyz="-0.0025002293460745202 0.0050800946525636995 0.0891495725401176" rpy="0 0 0"/>
+    <origin xyz="-0.0025002293460744717 0.006897943069782683 0.08902750816127794" rpy="0 0 0"/>
     <mass value="0.15062120277990856"/>
-    <inertia ixx="0.0005" iyy="0.000431" izz="6.9e-05" ixy="0.0" iyz="4e-06" ixz="0.0"/>
-  </inertial>
-  <visual>
-    <origin xyz="0.00534 0.011165 -0.163691" rpy="0 0 0"/>
+    <inertia ixx="0.0005" iyy="0.000431" izz="6.9e-05" ixy="0.0" iyz="-4e-06" ixz="0.0"/>
+  </inertial>
+  <visual>
+    <origin xyz="0.00534 0.10007 -0.133278" rpy="0 0 0"/>
     <geometry>
       <mesh filename="package://robot_arm_description/meshes/arm2_1.stl" scale="0.001 0.001 0.001"/>
@@ -178,5 +178,5 @@
   </visual>
   <collision>
-    <origin xyz="0.00534 0.011165 -0.163691" rpy="0 0 0"/>
+    <origin xyz="0.00534 0.10007 -0.133278" rpy="0 0 0"/>
     <geometry>
       <mesh filename="package://robot_arm_description/meshes/arm2_1.stl" scale="0.001 0.001 0.001"/>
@@ -186,10 +186,10 @@
 <link name="motor_3_1">
   <inertial>
-    <origin xyz="-0.014069306671155678 0.02862636241498935 0.0002871907251089101" rpy="0 0 0"/>
+    <origin xyz="-0.014069306671155623 0.028626500748401534 -0.00029710861420650936" rpy="0 0 0"/>
     <mass value="0.8439665579832097"/>
-    <inertia ixx="0.000579" iyy="0.000343" izz="0.000355" ixy="-0.0" iyz="-0.0" ixz="0.0"/>
-  </inertial>
-  <visual>
-    <origin xyz="0.01034 0.035656 -0.303045" rpy="0 0 0"/>
+    <inertia ixx="0.000579" iyy="0.000343" izz="0.000355" ixy="-0.0" iyz="0.0" ixz="0.0"/>
+  </inertial>
+  <visual>
+    <origin xyz="0.01034 0.121713 -0.273103" rpy="0 0 0"/>
     <geometry>
       <mesh filename="package://robot_arm_description/meshes/motor_3_1.stl" scale="0.001 0.001 0.001"/>
@@ -198,5 +198,5 @@
   </visual>
   <collision>
-    <origin xyz="0.01034 0.035656 -0.303045" rpy="0 0 0"/>
+    <origin xyz="0.01034 0.121713 -0.273103" rpy="0 0 0"/>
     <geometry>
       <mesh filename="package://robot_arm_description/meshes/motor_3_1.stl" scale="0.001 0.001 0.001"/>
@@ -206,10 +206,10 @@
 <link name="outaxis3_1">
   <inertial>
-    <origin xyz="0.004045016512819107 2.129035144363134e-07 2.4997477449106853e-07" rpy="0 0 0"/>
+    <origin xyz="0.004045016512819159 -2.557173771899901e-07 3.5961280409058105e-07" rpy="0 0 0"/>
     <mass value="0.03958817250937558"/>
     <inertia ixx="6e-06" iyy="3e-06" izz="3e-06" ixy="-0.0" iyz="0.0" ixz="-0.0"/>
   </inertial>
   <visual>
-    <origin xyz="0.01134 0.006658 -0.303355" rpy="0 0 0"/>
+    <origin xyz="0.01134 0.092714 -0.272821" rpy="0 0 0"/>
     <geometry>
       <mesh filename="package://robot_arm_description/meshes/outaxis3_1.stl" scale="0.001 0.001 0.001"/>
@@ -218,5 +218,5 @@
   </visual>
   <collision>
-    <origin xyz="0.01134 0.006658 -0.303355" rpy="0 0 0"/>
+    <origin xyz="0.01134 0.092714 -0.272821" rpy="0 0 0"/>
     <geometry>
       <mesh filename="package://robot_arm_description/meshes/outaxis3_1.stl" scale="0.001 0.001 0.001"/>
@@ -224,33 +224,22 @@
   </collision>
 </link>
-<link name="net_v1_1">
-  <inertial>
-    <origin xyz="0.007450286235457758 0.049310655974081664 0.15365933191011066" rpy="0 0 0"/>
+<link name="lacrosse_v1_1">
+  <inertial>
+    <origin xyz="0.007362943960072052 -0.15846473498340286 -0.01140236557371438" rpy="0 0 0"/>
     <mass value="0.10478191448055754"/>
-    <inertia ixx="0.009956" iyy="0.009892" izz="0.002412" ixy="-7e-06" iyz="-0.003105" ixz="-1.8e-05"/>
-  </inertial>
-  <visual>
-    <origin xyz="0.00334 -0.001927 -0.31174" rpy="0 0 0"/>
-    <geometry>
-      <mesh filename="package://robot_arm_description/meshes/net_1.stl" scale="0.001 0.001 0.001"/>
-    </geometry>
-    <material name="silver"/>
-  </visual>
-  <collision>
-    <origin xyz="0.00334 -0.001927 -0.31174" rpy="0 0 0"/>
-    <geometry>
-      <mesh filename="package://robot_arm_description/meshes/net_1.stl" scale="0.001 0.001 0.001"/>
-    </geometry>
-    <surface>
-      <friction>
-        <ode>
-          <mu>1</mu>       <!-- 摩擦系数 -->
-          <mu2>1</mu2>     <!-- 第二摩擦系数 -->
-        </ode>
-      </friction>
-      <bounce>
-        <restitution coefficient="0"/>  <!-- 恢复系数 -->
-      </bounce>
-    </surface>
+    <inertia ixx="0.000904" iyy="0.000121" izz="0.001006" ixy="2e-06" iyz="-2.6e-05" ixz="0.0"/>
+  </inertial>
+  <visual>
+    <origin xyz="0.00354 0.082813 -0.279601" rpy="0 0 0"/>
+    <geometry>
+      <mesh filename="package://robot_arm_description/meshes/lacrosse_v1_1.stl" scale="0.001 0.001 0.001"/>
+    </geometry>
+    <material name="silver"/>
+  </visual>
+  <collision>
+    <origin xyz="0.00354 0.082813 -0.279601" rpy="0 0 0"/>
+    <geometry>
+      <mesh filename="package://robot_arm_description/meshes/lacrosse_v1_1.stl" scale="0.001 0.001 0.001"/>
+    </geometry>
   </collision>
 </link>
@@ -266,5 +255,5 @@
 </joint>
 <joint name="Revolute2" type="continuous">
-  <origin xyz="-0.001 0.0 -0.029" rpy="0 0 0"/>
+  <origin xyz="-0.001 0.0 -0.029" rpy="-1 0 0"/>
   <parent link="motor_1_1"/>
   <child link="outaxis1_1"/>
@@ -272,5 +261,5 @@
 </joint>
 <joint name="Rigid3" type="fixed">
-  <origin xyz="0.008 -0.005889 -0.010456" rpy="0 0 0"/>
+  <origin xyz="0.008 0.001507 -0.011905" rpy="0 0 0"/>
   <parent link="outaxis1_1"/>
   <child link="fl1_1"/>
@@ -282,16 +271,16 @@
 </joint>
 <joint name="Rigid5" type="fixed">
-  <origin xyz="0.005 -0.024713 0.160138" rpy="0 0 0"/>
+  <origin xyz="0.005 -0.115322 0.113822" rpy="0 0 0"/>
   <parent link="arm1_1"/>
   <child link="motor_2_1"/>
 </joint>
 <joint name="Revolute6" type="continuous">
-  <origin xyz="0.001 0.028998 0.00031" rpy="0 0 0"/>
+  <origin xyz="0.001 0.023094 0.017539" rpy="1 0 0"/>
   <parent link="motor_2_1"/>
   <child link="outaxis2_1"/>
-  <axis xyz="-1.0 -0.0 -0.0"/>
+  <axis xyz="1.0 -0.0 -0.0"/>
 </joint>
 <joint name="Rigid7" type="fixed">
-  <origin xyz="-0.008 -0.006111 0.010327" rpy="0 0 0"/>
+  <origin xyz="-0.008 -0.005899 0.01045" rpy="0 0 0"/>
   <parent link="outaxis2_1"/>
   <child link="fl2_1"/>
@@ -303,18 +292,18 @@
 </joint>
 <joint name="Rigid9" type="fixed">
-  <origin xyz="-0.005 -0.024491 0.139354" rpy="0 0 0"/>
+  <origin xyz="-0.005 -0.021643 0.139825" rpy="0 0 0"/>
   <parent link="arm2_1"/>
   <child link="motor_3_1"/>
 </joint>
 <joint name="Revolute10" type="continuous">
-  <origin xyz="-0.001 0.028998 0.00031" rpy="0 0 0"/>
+  <origin xyz="0.001 0.028999 -0.000282" rpy="-1 0 0"/>
   <parent link="motor_3_1"/>
   <child link="outaxis3_1"/>
   <axis xyz="1.0 0.0 0.0"/>
 </joint>
-<joint name="Rigid11" type="fixed">
-  <origin xyz="0.008 0.008585 0.008385" rpy="0 0 0"/>
+<joint name="Rigid13" type="fixed">
+  <origin xyz="0.01 -0.009901 0.001" rpy="0 0 0"/>
   <parent link="outaxis3_1"/>
-  <child link="net_v1_1"/>
+  <child link="lacrosse_v1_1"/>
 </joint>
 </robot>
